File: KiCad/Easy-PCB.sch (KiCad schematic (older format))
At the start: 20 parts, among them J1 IEC Male Inlet: 703W-00/53, J3 HLW20R-2C7LF, P1 Molex 0022032021, P2 Molex 0901200126, P3 Molex 0022032041, P4 Molex 387203208, P5 Molex 0022032021, Q1 2N3904, SW1 SPST: DF62J12S2AHQA, U1 PIC16F883

Commit message: kicad resistor package associations complete
Parts:
- R10, R11, R12, R13, R14, R15, R9: footprint (none) -> Resistors_ThroughHole:Resistor_Horizontal_RM10mm
- RP1: footprint (none) -> Buttons_Switches_ThroughHole:SW_DIP_x8_Slide
Changed lines of the file:
@@
 F 0 "R11" V 5380 2050 50  0000 C CNN
 F 1 "10k" V 5300 2050 50  0000 C CNN
-F 2 "" V 5230 2050 50  0001 C CNN
+F 2 "Resistors_ThroughHole:Resistor_Horizontal_RM10mm" V 5230 2050 50  0001 C CNN
 F 3 "" H 5300 2050 50  0000 C CNN
 	1    5300 2050
@@
 F 0 "R12" V 5680 2050 50  0000 C CNN
 F 1 "10k" V 5600 2050 50  0000 C CNN
-F 2 "" V 5530 2050 50  0001 C CNN
+F 2 "Resistors_ThroughHole:Resistor_Horizontal_RM10mm" V 5530 2050 50  0001 C CNN
 F 3 "" H 5600 2050 50  0000 C CNN
 	1    5600 2050
@@
 F 0 "R13" V 5980 2050 50  0000 C CNN
 F 1 "10k" V 5900 2050 50  0000 C CNN
-F 2 "" V 5830 2050 50  0001 C CNN
+F 2 "Resistors_ThroughHole:Resistor_Horizontal_RM10mm" V 5830 2050 50  0001 C CNN
 F 3 "" H 5900 2050 50  0000 C CNN
 	1    5900 2050
@@
 F 0 "R10" V 3380 5500 50  0000 C CNN
 F 1 "10k" V 3300 5500 50  0000 C CNN
-F 2 "" V 3230 5500 50  0001 C CNN
+F 2 "Resistors_ThroughHole:Resistor_Horizontal_RM10mm" V 3230 5500 50  0001 C CNN
 F 3 "" H 3300 5500 50  0000 C CNN
 	1    3300 5500
@@
 F 0 "R15" V 8580 3950 50  0000 C CNN
 F 1 "1k" V 8500 3950 50  0000 C CNN
-F 2 "" V 8430 3950 50  0001 C CNN
+F 2 "Resistors_ThroughHole:Resistor_Horizontal_RM10mm" V 8430 3950 50  0001 C CNN
 F 3 "" H 8500 3950 50  0000 C CNN
 	1    8500 3950
@@
 F 0 "R14" V 8330 4350 50  0000 C CNN
 F 1 "1k" V 8250 4350 50  0000 C CNN
-F 2 "" V 8180 4350 50  0001 C CNN
+F 2 "Resistors_ThroughHole:Resistor_Horizontal_RM10mm" V 8180 4350 50  0001 C CNN
 F 3 "" H 8250 4350 50  0000 C CNN
 	1    8250 4350
@@
 F 0 "R9" V 2050 4700 50  0000 C CNN
 F 1 "1k" V 2100 4500 50  0000 C CNN
-F 2 "" V 2030 4500 50  0001 C CNN
+F 2 "Resistors_ThroughHole:Resistor_Horizontal_RM10mm" V 2030 4500 50  0001 C CNN
 F 3 "" H 2100 4500 50  0000 C CNN
 	1    2100 4500
@@
 F 0 "RP1" H 1800 4400 50  0000 C CNN
 F 1 "320" H 1800 3500 50  0000 C CNN
-F 2 "" H 1800 3950 50  0001 C CNN
+F 2 "Buttons_Switches_ThroughHole:SW_DIP_x8_Slide" H 1800 3950 50  0001 C CNN
 F 3 "" H 1800 3950 50  0000 C CNN
 	1    1800 3950

Commit message: capacitors and diode part associations
Parts:
- C1: footprint (none) -> Capacitors_ThroughHole:C_Disc_D3_P2.5
- J3: footprint (none) -> Easy-PCB-footprints:HLW20R-2C7LF
Changed lines of the file:
@@
 F 0 "J3" H 1000 4700 50  0000 C CNN
 F 1 "HLW20R-2C7LF" V 1100 3650 50  0000 C CNN
-F 2 "" H 1000 3650 60  0001 C CNN
+F 2 "Easy-PCB-footprints:HLW20R-2C7LF" H 1000 3650 60  0001 C CNN
 F 3 "" H 1000 3650 60  0000 C CNN
 	1    1000 3650
@@
 F 0 "C1" H 1710 3320 50  0000 L CNN
 F 1 "0.1u" H 1710 3170 50  0000 L CNN
-F 2 "" H 1700 3250 50  0001 C CNN
+F 2 "Capacitors_ThroughHole:C_Disc_D3_P2.5" H 1700 3250 50  0001 C CNN
 F 3 "" H 1700 3250 50  0000 C CNN
 	1    1700 3250

Commit message: IC BOM and footprints complete
Parts:
- removed Q1: 2N3904, symbol MMBT3904
- added Q1: 2N3904, Easy-PCB-footprints:TO-92, symbol 2N3904
- J1: value IEC Male Inlet: 703W-00/53 -> 703W-00/53
- SW1: value SPST: DF62J12S2AHQA -> DF62J12S2AHQA
- U1: footprint (none) -> Easy-PCB-footprints:DIP-28
Connections:
- net GND: now also Q1.1 (E)
- net at R15.2, SP1.2: now also Q1.3 (C)
- net at R14.1: now also Q1.2 (B)
Changed lines of the file:
@@
 F 0 "U1" H 4050 3450 60  0000 C CNN
 F 1 "PIC16F883" H 4050 3550 60  0000 C CNN
-F 2 "" H 4050 3600 60  0001 C CNN
+F 2 "Easy-PCB-footprints:DIP-28" H 4050 3600 60  0001 C CNN
 F 3 "" H 4050 3600 60  0000 C CNN
 	1    4050 3600
@@
 $EndComp
 $Comp
-L MMBT3904 Q1
-U 1 1 56815FFA
-P 8600 4350
-F 0 "Q1" H 8800 4425 50  0000 L CNN
-F 1 "2N3904" H 8800 4350 50  0000 L CNN
-F 2 "" H 8800 4275 50  0001 L CIN
-F 3 "" H 8600 4350 50  0000 L CNN
-	1    8600 4350
-	1    0    0    -1
-$EndComp
-$Comp
 L R R15
 U 1 1 56816949
@@
 U 1 1 56821A1C
 P 6700 1300
-F 0 "J1" H 7700 1400 60  0000 C CNN
-F 1 "IEC Male Inlet: 703W-00/53" H 7700 1300 60  0000 C CNN
+F 0 "J1" H 7350 1400 60  0000 C CNN
+F 1 "703W-00/53" H 7350 1300 60  0000 C CNN
 F 2 "" H 6700 1300 60  0001 C CNN
 F 3 "" H 6700 1300 60  0000 C CNN
@@
 P 7750 2050
 F 0 "SW1" H 7750 2250 50  0000 C CNN
-F 1 "SPST: DF62J12S2AHQA" H 7750 1900 50  0000 C CNN
+F 1 "DF62J12S2AHQA" H 7750 1900 50  0000 C CNN
 F 2 "" H 7750 2050 50  0001 C CNN
 F 3 "" H 7750 2050 50  0000 C CNN
@@
 Wire Wire Line
 	6500 4000 6750 4000
+$Comp
+L 2N3904 Q1
+U 1 1 56880FA0
+P 8600 4350
+F 0 "Q1" H 8800 4425 50  0000 L CNN
+F 1 "2N3904" H 8800 4350 50  0000 L CNN
+F 2 "Easy-PCB-footprints:TO-92" H 8800 4275 50  0000 L CIN
+F 3 "" H 8600 4350 50  0000 L CNN
+	1    8600 4350
+	1    0    0    -1
+$EndComp
 $EndSCHEMATC
