File: KiCad/Easy-PCB.sch (KiCad schematic (older format))
At the start: 27 parts, among them J1 703W-00/53, J3 HLW20R-2C7LF, P1 1x02, P10 via, P11 via, P13 via, P2 1x06, P3 1x04, P4 1x03 Terminal Block, P5 1x02, P6 via, P7 via, P8 via, P9 via, Q1 2N3904, SW1 R1966ABLKBLKFR, U1 PIC16F883

Commit message: routing complete
Parts:
- added P14, P15, P16, P17, P18, P19: via, Connect:PINTST, symbol CONN_01X01
Connections:
- net GND: now also P14.1 (P1), P15.1 (P1), P17.1 (P1), P18.1 (P1)
- net Reset: now reaches P2.1 (P1), R10.2, R9.1, U1.1 (RE3/~MCLR~/Vpp)
- net Reset: now also P19.1 (P1)
- net Motor Driver/Motor_On renamed Motor_On
- net Motor_On: now also P16.1 (P1)
Changed lines of the file:
@@
 Text GLabel 2475 6775 1    60   Input ~ 0
 CS2
+$Comp
+L CONN_01X01 P14
+U 1 1 56A2BF77
+P 2700 7050
+F 0 "P14" H 2700 7150 50  0000 C CNN
+F 1 "via" V 2800 7050 50  0000 C CNN
+F 2 "Connect:PINTST" H 2700 7050 50  0001 C CNN
+F 3 "" H 2700 7050 50  0000 C CNN
+	1    2700 7050
+	0    1    1    0
+$EndComp
+$Comp
+L GND #PWR016
+U 1 1 56A2C3C6
+P 2700 6775
+F 0 "#PWR016" H 2700 6525 50  0001 C CNN
+F 1 "GND" H 2700 6625 50  0000 C CNN
+F 2 "" H 2700 6775 50  0000 C CNN
+F 3 "" H 2700 6775 50  0000 C CNN
+	1    2700 6775
+	-1   0    0    1
+$EndComp
+Wire Wire Line
+	2700 6775 2700 6850
+$Comp
+L CONN_01X01 P15
+U 1 1 56A2CB3C
+P 2925 7050
+F 0 "P15" H 2925 7150 50  0000 C CNN
+F 1 "via" V 3025 7050 50  0000 C CNN
+F 2 "Connect:PINTST" H 2925 7050 50  0001 C CNN
+F 3 "" H 2925 7050 50  0000 C CNN
+	1    2925 7050
+	0    1    1    0
+$EndComp
+$Comp
+L GND #PWR017
+U 1 1 56A2CCE5
+P 2925 6775
+F 0 "#PWR017" H 2925 6525 50  0001 C CNN
+F 1 "GND" H 2925 6625 50  0000 C CNN
+F 2 "" H 2925 6775 50  0000 C CNN
+F 3 "" H 2925 6775 50  0000 C CNN
+	1    2925 6775
+	-1   0    0    1
+$EndComp
+Wire Wire Line
+	2925 6850 2925 6775
+$Comp
+L CONN_01X01 P16
+U 1 1 56A2EBBC
+P 3150 7050
+F 0 "P16" H 3150 7150 50  0000 C CNN
+F 1 "via" V 3250 7050 50  0000 C CNN
+F 2 "Connect:PINTST" H 3150 7050 50  0001 C CNN
+F 3 "" H 3150 7050 50  0000 C CNN
+	1    3150 7050
+	0    1    1    0
+$EndComp
+Wire Wire Line
+	3150 6850 3150 6775
+Text GLabel 3150 6775 1    60   Input ~ 0
+Motor_On
+Text GLabel 8200 3200 3    60   Input ~ 0
+Motor_On
+$Comp
+L CONN_01X01 P17
+U 1 1 56A305FB
+P 3375 7050
+F 0 "P17" H 3375 7150 50  0000 C CNN
+F 1 "via" V 3475 7050 50  0000 C CNN
+F 2 "Connect:PINTST" H 3375 7050 50  0001 C CNN
+F 3 "" H 3375 7050 50  0000 C CNN
+	1    3375 7050
+	0    1    1    0
+$EndComp
+Wire Wire Line
+	3375 6850 3375 6775
+$Comp
+L GND #PWR018
+U 1 1 56A308A6
+P 3375 6775
+F 0 "#PWR018" H 3375 6525 50  0001 C CNN
+F 1 "GND" H 3375 6625 50  0000 C CNN
+F 2 "" H 3375 6775 50  0000 C CNN
+F 3 "" H 3375 6775 50  0000 C CNN
+	1    3375 6775
+	-1   0    0    1
+$EndComp
+$Comp
+L CONN_01X01 P18
+U 1 1 56A31D71
+P 3600 7050
+F 0 "P18" H 3600 7150 50  0000 C CNN
+F 1 "via" V 3700 7050 50  0000 C CNN
+F 2 "Connect:PINTST" H 3600 7050 50  0001 C CNN
+F 3 "" H 3600 7050 50  0000 C CNN
+	1    3600 7050
+	0    1    1    0
+$EndComp
+Wire Wire Line
+	3600 6850 3600 6775
+$Comp
+L GND #PWR019
+U 1 1 56A32319
+P 3600 6775
+F 0 "#PWR019" H 3600 6525 50  0001 C CNN
+F 1 "GND" H 3600 6625 50  0000 C CNN
+F 2 "" H 3600 6775 50  0000 C CNN
+F 3 "" H 3600 6775 50  0000 C CNN
+	1    3600 6775
+	-1   0    0    1
+$EndComp
+Text GLabel 4025 5700 1    60   Input ~ 0
+Reset
+$Comp
+L CONN_01X01 P19
+U 1 1 56A33F66
+P 3825 7050
+F 0 "P19" H 3825 7150 50  0000 C CNN
+F 1 "via" V 3925 7050 50  0000 C CNN
+F 2 "Connect:PINTST" H 3825 7050 50  0001 C CNN
+F 3 "" H 3825 7050 50  0000 C CNN
+	1    3825 7050
+	0    1    1    0
+$EndComp
+Wire Wire Line
+	3825 6850 3825 6775
+Text GLabel 3825 6775 1    60   Input ~ 0
+Reset
 $EndSCHEMATC
