File: KiCad/Motor-Driver.sch (KiCad schematic (older format))
At the start: 38 parts, among them Q10 MJE350, Q11 2N3904, Q12 2N3904, Q13 MJE340, Q14 MJE350, Q15 2N3904, Q16 MJE340, Q17 MJE350, Q18 2N3904, Q3 2N3904, Q4 2N3904, Q5 MJE340, Q6 MJE350, Q7 2N3904, Q8 2N3904, Q9 MJE340

Commit message: footprint associations complete
Parts:
- Q10, Q13, Q14, Q16, Q17, Q5, Q6, Q9: footprint (none) -> Easy-PCB-footprints:MJE3x0
Changed lines of the file:
@@
 F 0 "Q9" H 4700 2175 50  0000 L CNN
 F 1 "MJE340" H 4700 2100 50  0000 L CNN
-F 2 "" H 4700 2025 50  0001 L CIN
+F 2 "Easy-PCB-footprints:MJE3x0" H 4700 2025 50  0001 L CIN
 F 3 "" H 4500 2100 50  0000 L CNN
 	1    4500 2100
@@
 F 0 "Q13" H 6600 2175 50  0000 L CNN
 F 1 "MJE340" H 6600 2100 50  0000 L CNN
-F 2 "" H 6600 2025 50  0001 L CIN
+F 2 "Easy-PCB-footprints:MJE3x0" H 6600 2025 50  0001 L CIN
 F 3 "" H 6400 2100 50  0000 L CNN
 	1    6400 2100
@@
 F 0 "Q16" H 8500 2175 50  0000 L CNN
 F 1 "MJE340" H 8500 2100 50  0000 L CNN
-F 2 "" H 8500 2025 50  0001 L CIN
+F 2 "Easy-PCB-footprints:MJE3x0" H 8500 2025 50  0001 L CIN
 F 3 "" H 8300 2100 50  0000 L CNN
 	1    8300 2100
@@
 F 0 "Q5" H 2800 2175 50  0000 L CNN
 F 1 "MJE340" H 2800 2100 50  0000 L CNN
-F 2 "" H 2800 2025 50  0001 L CIN
+F 2 "Easy-PCB-footprints:MJE3x0" H 2800 2025 50  0001 L CIN
 F 3 "" H 2600 2100 50  0000 L CNN
 	1    2600 2100
@@
 F 0 "Q6" H 2800 3675 50  0000 L CNN
 F 1 "MJE350" H 2800 3600 50  0000 L CNN
-F 2 "" H 2800 3525 50  0001 L CIN
+F 2 "Easy-PCB-footprints:MJE3x0" H 2800 3525 50  0001 L CIN
 F 3 "" H 2600 3600 50  0000 L CNN
 	1    2600 3600
@@
 F 0 "Q10" H 4700 3675 50  0000 L CNN
 F 1 "MJE350" H 4700 3600 50  0000 L CNN
-F 2 "" H 4700 3525 50  0001 L CIN
+F 2 "Easy-PCB-footprints:MJE3x0" H 4700 3525 50  0001 L CIN
 F 3 "" H 4500 3600 50  0000 L CNN
 	1    4500 3600
@@
 F 0 "Q14" H 6600 3675 50  0000 L CNN
 F 1 "MJE350" H 6600 3600 50  0000 L CNN
-F 2 "" H 6600 3525 50  0001 L CIN
+F 2 "Easy-PCB-footprints:MJE3x0" H 6600 3525 50  0001 L CIN
 F 3 "" H 6400 3600 50  0000 L CNN
 	1    6400 3600
@@
 F 0 "Q17" H 8500 3675 50  0000 L CNN
 F 1 "MJE350" H 8500 3600 50  0000 L CNN
-F 2 "" H 8500 3525 50  0001 L CIN
+F 2 "Easy-PCB-footprints:MJE3x0" H 8500 3525 50  0001 L CIN
 F 3 "" H 8300 3600 50  0000 L CNN
 	1    8300 3600
